File: Hardware/Dieguito Regleta/Regleta16_V1.kicad_pcb (KiCad board)
At the start: 2 copper layers, 124.4 x 46.6 mm, 46 parts, among them J2 Conn_01x07, U1 QRE1113GR, U10 QRE1113GR, U11 QRE1113GR, U12 QRE1113GR, U13 QRE1113GR, U14 QRE1113GR, U15 QRE1113GR, U16 QRE1113GR, U18 CD74HC4067M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

Commit message: Subo carpetas
Parts:
- added G***: LOGO, Library:firma_diego, B.Cu at (137.2, 68.7)
