File: Hardware/Dieguito Main/Dieguito.kicad_sch (KiCad schematic)
At the start: 39 parts, among them J1 XT30, J2 Cable_PAD, J3 Cable_PAD, J4 Programador, J5 Sensores, J6 Turbina, Q1 AO3400A, SW1 ENABLE, SW2 BOOT, SW3 GO/STOP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

Commit message: Actualizo Hardware
Changed lines of the file:
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@@
+	(wire
+		(pts
+			(xy 85.09 96.52) (xy 86.36 96.52)
+		)
+		(stroke
+			(width 0)
+			(type default)
+		)
+	)
 	(wire
 		(pts
@@
 	(global_label "LED"
 		(shape input)
-		(at 86.36 96.52 180)
-		(fields_autoplaced yes)
-		(effects
-			(font
-				(size 1.27 1.27)
-			)
-			(justify right)
-		)
-		(property "Intersheetrefs" "${INTERSHEET_REFS}"
-			(at 79.9277 96.52 0)
-			(effects
-				(font
+		(at 85.09 96.52 180)
+		(fields_autoplaced yes)
+		(effects
+			(font
+				(size 1.27 1.27)
+			)
+			(justify right)
+		)
+		(property "Intersheetrefs" "${INTERSHEET_REFS}"
+			(at 78.6577 96.52 0)
+			(effects
+				(font

Commit message: Actualizo carpetas
Parts:
- removed J4: Programador, Connector_PinSocket_2.54mm:PinSocket_1x04_P2.54mm_Vertical, symbol Connector_Generic:Conn_01x04
- added J4: Programador, Connector_PinSocket_2.54mm:PinSocket_1x05_P2.54mm_Vertical, symbol Connector_Generic:Conn_01x05
Connections:
- net +3.3V: now also J4.2 (Pin_2)
- net +5V: now also J4.1 (Pin_1)
- net GND: now also J4.5 (Pin_5)
- net RXD0: now also J4.4 (Pin_4)
- net TXD0: now also J4.3 (Pin_3)
Changed lines of the file:
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@@
 	(wire
 		(pts
-			(xy 213.36 128.27) (xy 217.17 128.27)
+			(xy 209.55 128.27) (xy 217.17 128.27)
 		)
 		(stroke
@@
 	(wire
 		(pts
+			(xy 214.63 125.73) (xy 217.17 125.73)
+		)
+		(stroke
+			(width 0)
+			(type default)
+		)
+	)
+	(wire
+		(pts
 			(xy 214.63 38.1) (xy 214.63 45.72)
 		)
@@
 	(symbol
 		(lib_id "power:+3.3V")
-		(at 213.36 128.27 0)
+		(at 209.55 128.27 0)
 		(unit 1)
 		(exclude_from_sim no)
@@
 		(fields_autoplaced yes)
 		(property "Reference" "#PWR017"
-			(at 213.36 132.08 0)
+			(at 209.55 132.08 0)
 			(effects
 				(font
@@
 		)
 		(property "Value" "+3.3V"
-			(at 213.36 123.19 0)
+			(at 209.55 123.19 0)
 			(effects
 				(font
@@
 		)
 		(property "Footprint" ""
-			(at 213.36 128.27 0)
+			(at 209.55 128.27 0)
 			(effects
 				(font
@@
 		)
 		(property "Datasheet" ""
-			(at 213.36 128.27 0)
+			(at 209.55 128.27 0)
 			(effects
 				(font
@@
 		)
 		(property "Description" "Power symbol creates a global label with name \"+3.3V\""
-			(at 213.36 128.27 0)
+			(at 209.55 128.27 0)
 			(effects
 				(font
@@
 	)
 	(symbol
+		(lib_id "Connector_Generic:Conn_01x05")
+		(at 222.25 130.81 0)
+		(unit 1)
+		(exclude_from_sim no)
+		(in_bom yes)
+		(on_board yes)
+		(dnp no)
+		(fields_autoplaced yes)
+		(property "Reference" "J4"
+			(at 224.79 129.5399 0)
+			(effects
+				(font
+					(size 1.27 1.27)
+				)
+				(justify left)
+			)
+		)
+		(property "Value" "Programador"
+			(at 224.79 132.0799 0)
+			(effects
+				(font
+					(size 1.27 1.27)
+				)
+				(justify left)
+			)
+		)
+		(property "Footprint" "Connector_PinSocket_2.54mm:PinSocket_1x05_P2.54mm_Vertical"
+			(at 222.25 130.81 0)
+			(effects
+				(font
+					(size 1.27 1.27)
+				)
+				(hide yes)
+			)
+		)
+		(property "Datasheet" "~"
+			(at 222.25 130.81 0)
+			(effects
+				(font
+					(size 1.27 1.27)
+				)
+				(hide yes)
+			)
+		)
+		(property "Description" "Generic connector, single row, 01x05, script generated (kicad-library-utils/schlib/autogen/connector/)"
+			(at 222.25 130.81 0)
+			(effects
+				(font
+					(size 1.27 1.27)
+				)
+				(hide yes)
+			)
+		)
+		(pin "1"
+		)
+		(pin "5"
+		)
+		(pin "2"
+		)
+		(pin "3"
+		)
+		(pin "4"
+		)
+		(instances
+			(project ""
+				(path "/e7d1ffde-f2af-4684-b5b5-9911fccaf4fa"
+					(reference "J4")
+					(unit 1)
+				)
+			)
+		)
+	)
+	(symbol
 		(lib_id "Device:R")
 		(at 90.17 74.93 90)
@@
 	)
 	(symbol
-		(lib_id "Connector_Generic:Conn_01x04")
-		(at 222.25 130.81 0)
-		(unit 1)
-		(exclude_from_sim no)
-		(in_bom yes)
-		(on_board yes)
-		(dnp no)
-		(fields_autoplaced yes)
-		(property "Reference" "J4"
-			(at 224.79 130.8099 0)
-			(effects
-				(font
-					(size 1.27 1.27)
-				)
-				(justify left)
-			)
-		)
-		(property "Value" "Programador"
-			(at 224.79 133.3499 0)
-			(effects
-				(font
-					(size 1.27 1.27)
-				)
-				(justify left)
-			)
-		)
-		(property "Footprint" "Connector_PinSocket_2.54mm:PinSocket_1x04_P2.54mm_Vertical"
-			(at 222.25 130.81 0)
-			(effects
-				(font
-					(size 1.27 1.27)
-				)
-				(hide yes)
-			)
-		)
-		(property "Datasheet" "~"
-			(at 222.25 130.81 0)
-			(effects
-				(font
-					(size 1.27 1.27)
-				)
-				(hide yes)
-			)
-		)
-		(property "Description" "Generic connector, single row, 01x04, script generated (kicad-library-utils/schlib/autogen/connector/)"
-			(at 222.25 130.81 0)
-			(effects
-				(font
-					(size 1.27 1.27)
-				)
-				(hide yes)
-			)
-		)
-		(pin "1"
-		)
-		(pin "3"
-		)
-		(pin "4"
-		)
-		(pin "2"
-		)
-		(instances
-			(project ""
-				(path "/e7d1ffde-f2af-4684-b5b5-9911fccaf4fa"
-					(reference "J4")
-					(unit 1)
-				)
-			)
-		)
-	)
-	(symbol
 		(lib_id "Device:C")
 		(at 219.71 45.72 90)
@@
 					(unit 1)
 				)
+			)
+		)
+	)
+	(symbol
+		(lib_id "power:+5V")
+		(at 214.63 125.73 0)
+		(unit 1)
+		(exclude_from_sim no)
+		(in_bom yes)
+		(on_board yes)
+		(dnp no)
+		(property "Reference" "#PWR030"
+			(at 214.63 129.54 0)
+			(effects
+				(font
+					(size 1.27 1.27)
+				)
+				(hide yes)
+			)
+		)
+		(property "Value" "+5V"
+			(at 214.63 121.412 0)
+			(effects
+				(font
+					(size 1.27 1.27)
+				)
+			)
+		)
+		(property "Footprint" ""
+			(at 214.63 125.73 0)
+			(effects
+				(font
+					(size 1.27 1.27)
+				)
+				(hide yes)
+			)
+		)
+		(property "Datasheet" ""
+			(at 214.63 125.73 0)
+			(effects
+				(font
+					(size 1.27 1.27)
+				)
+				(hide yes)
+			)
+		)
+		(property "Description" "Power symbol creates a global label with name \"+5V\""
+			(at 214.63 125.73 0)
+			(effects
+				(font
+					(size 1.27 1.27)
+				)
+				(hide yes)
+			)
+		)
+		(pin "1"
+		)
+		(instances
+			(project "Dieguito"
+				(path "/e7d1ffde-f2af-4684-b5b5-9911fccaf4fa"
+					(reference "#PWR030")
+					(unit 1)
+				)

Commit message: Correcion de placa
Parts:
- removed C2, C3: 100u, Capacitor_SMD:C_Elec_6.3x7.7, symbol Device:C_Polarized
- added C2, C3: 10u, Capacitor_SMD:C_0805_2012Metric_Pad1.18x1.45mm_HandSolder, symbol Device:C
Connections:
- net +3.3V: now also C3.1
- net +5V: now also C2.1
- net AI1: now also U2.11 (IO26); no longer U2.9 (IO33)
- net AI2: now also U2.12 (IO27); no longer U2.8 (IO32)
- net BI1: now also U2.9 (IO33); no longer U2.11 (IO26)
- net BI2: now also U2.8 (IO32); no longer U2.12 (IO27)
- net GND: now also C2.2, C3.2
- net PWMA: now also U2.36 (IO22); no longer U2.33 (IO21)
- net PWMB: now also U2.33 (IO21); no longer U2.36 (IO22)
- net VCC: no longer U1.1 (VM)
- net at C7.1, U1.4 (A01): now also J2.2; no longer J2.1
- net at C7.2, U1.5 (A02): now also J2.1; no longer J2.2
- net at C8.2, U1.6 (B02): now also J3.1; no longer J3.2
- net at C8.1, U1.7 (B01): now also J3.2; no longer J3.1
- net VM: now reaches J1.2 (Pin_2), SW4.2 (B)
- net VM: now also U1.1 (VM)
