File: Hardware/Dieguito Main/Dieguito.kicad_pcb (KiCad board)
At the start: 2 copper layers, 124.4 x 79.8 mm, 46 parts, among them J1 XT30, J2 Cable_PAD, J3 Cable_PAD, J4 Programador, J5 Sensores, J6 Turbina, Q1 AO3400A, SW4 SW_SPDT, U1 ROB-14450, U2 ESP32-WROOM-32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

Commit message: Actualizo Hardware
Parts:
- renumbered D2 to ESP, D1 to LED, D3 to POWER
Routing:
- net VCC: track 78.2 -> 79.3 mm
- net D23: track 41.3 -> 42.2 mm
- net PWMB: track 27.2 -> 27.8 mm
- net GND: vias 13 -> 21

Commit message: Actualizo carpetas
Parts:
- J4: footprint Connector_PinSocket_2.54mm:PinSocket_1x04_P2.54mm_Vertical -> Connector_PinSocket_2.54mm:PinSocket_1x05_P2.54mm_Vertical
Connections:
- J4 pad 1: +3.3V -> +5V
- J4 pad 2: TXD0 -> +3.3V
- J4 pad 3: RXD0 -> TXD0
- J4 pad 4: GND -> RXD0
Routing:
- net +5V: track 111.0 -> 157.8 mm, vias 5 -> 8
- net RXD0: track 39.9 -> 42.3 mm
- net +3.3V: track 164.7 -> 164.2 mm

Commit message: Correcion de placa
Parts:
- removed BOOT: BOOT, Button_Switch_SMD:SW_Push_1P1T_NO_CK_KMR2
- removed EN: ENABLE, Button_Switch_SMD:SW_Push_1P1T_NO_CK_KMR2
- removed ESP, LED, POWER: POWER, LED_SMD:LED_0805_2012Metric_Pad1.15x1.40mm_HandSolder
- removed GO/STOP: GO/STOP, Button_Switch_SMD:SW_Push_1P1T_NO_CK_KMR2
- added D1: POWER, LED_SMD:LED_0805_2012Metric_Pad1.15x1.40mm_HandSolder, F.Cu at (250.8, 104.7)
- added D2: POWER, LED_SMD:LED_0805_2012Metric_Pad1.15x1.40mm_HandSolder, F.Cu at (256.6, 104.7)
- added D3: POWER, LED_SMD:LED_0805_2012Metric_Pad1.15x1.40mm_HandSolder, F.Cu at (245.0, 104.7)
- added SW1: ENABLE, Button_Switch_SMD:SW_Push_1P1T_NO_CK_KMR2, F.Cu at (157.9, 102.5)
- added SW2: BOOT, Button_Switch_SMD:SW_Push_1P1T_NO_CK_KMR2, F.Cu at (184.5, 102.3)
- added SW3: GO/STOP, Button_Switch_SMD:SW_Push_1P1T_NO_CK_KMR2, F.Cu at (153.1, 142.2)
- C2, C3: value 100u -> 10u; footprint Capacitor_SMD:C_Elec_6.3x7.7 -> Capacitor_SMD:C_0805_2012Metric_Pad1.18x1.45mm_HandSolder
- moved C9 89.7 mm to (252.5, 128.1)
- moved R8 78.0 mm to (248.6, 124.1), turned to 0 degrees
- moved D4 77.5 mm to (243.7, 128.1)
- moved Q1 76.6 mm to (248.6, 128.1)
- moved C3 73.1 mm to (238.3, 148.8), turned to 180 degrees
- moved R9 72.2 mm to (248.6, 132.7), turned to 180 degrees
- moved C4 67.4 mm to (238.3, 152.2), turned to 180 degrees
- moved C1 66.2 mm to (242.8, 148.9), turned to 0 degrees
- moved U3 64.9 mm to (240.4, 142.4), turned to 90 degrees
- moved J6 61.0 mm to (237.6, 129.2)
- moved C2 58.6 mm to (242.8, 152.3), turned to 0 degrees
- moved REF** 55.6 mm to (230.2, 109.6)
- moved REF** 55.5 mm to (190.8, 109.6)
- moved U1 40.1 mm to (171.6, 142.7), turned to 90 degrees
- moved REF** 38.7 mm to (190.8, 149.0)
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Connections:
- J1 pad 2: Net-(J1-Pin_2) -> /VM
- J2 pad 1: Net-(U1-A01) -> Net-(U1-A02)
- J2 pad 2: Net-(U1-A02) -> Net-(U1-A01)
- J3 pad 1: Net-(U1-B01) -> Net-(U1-B02)
- J3 pad 2: Net-(U1-B02) -> Net-(U1-B01)
- SW4 pad 2: Net-(J1-Pin_2) -> /VM
- U1 pad 1: VCC -> /VM
- U2 pad 11: BI1 -> AI1
- U2 pad 12: BI2 -> AI2
- U2 pad 33: PWMA -> PWMB
- U2 pad 36: PWMB -> PWMA
- U2 pad 8: AI2 -> BI2
- U2 pad 9: AI1 -> BI1
Routing:
- net /VM: track 0.00 -> 144.4 mm
- net +5V: track 157.8 -> 208.5 mm, vias 8 -> 5
- net LED: track 73.9 -> 116.0 mm, vias 0 -> 2
- net AI2: track 54.7 -> 15.1 mm
- net D23: track 42.2 -> 79.6 mm, vias 2 -> 4
- net Net-(U1-A02): track 69.5 -> 32.5 mm
- net Net-(J1-Pin_2): track 36.0 -> 0.00 mm, vias 2 -> 0
- net VCC: track 79.3 -> 45.3 mm
- net AI1: track 51.1 -> 18.0 mm
- net BI1: track 50.3 -> 24.4 mm
- net BI2: track 48.9 -> 26.6 mm
- net Net-(U1-A01): track 58.6 -> 39.1 mm
- net SIG: track 44.7 -> 60.4 mm
- net Net-(U1-B02): track 55.1 -> 68.7 mm
- net RXD0: track 42.3 -> 31.3 mm
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Other:
- board size 124.4 x 79.8 mm -> 124.4 x 91.3 mm

Commit message: Corrijo placa main
Parts:
- renumbered D2 to 3,3V, D3 to BATT, SW2 to BOOT, SW1 to EN, D1 to LED, SW3 to STOP/GO
Routing:
- net GND: vias 18 -> 19
Changed lines of the file:
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@@
 		(descr "LED SMD 0805 (2012 Metric), square (rectangular) end terminal, IPC-7351 nominal, (Body size source: https://docs.google.com/spreadsheets/d/1BsfQQcO9C6DZCsRaXUlFlo91Tg2WpOkGARC1WS5S8t0/edit?usp=sharing), generated with kicad-footprint-generator")
 		(tags "LED handsolder")
-		(property "Reference" "D1"
-			(at 0 -1.65 90)
+		(property "Reference" "LED"
+			(at -3.399801 0.0196 180)
 			(layer "F.SilkS")
 			(effects
@@
 			(at 0 1.65 90)
 			(layer "F.Fab")
+			(hide yes)
 			(effects
 				(font
@@
 		(descr "CK components KMR2 tactile switch http://www.ckswitches.com/media/1479/kmr2.pdf")
 		(tags "tactile switch kmr2")
-		(property "Reference" "SW2"
-			(at 0 -2.45 0)
+		(property "Reference" "BOOT"
+			(at 0.004799 -2.2594 0)
 			(layer "F.SilkS")
 			(effects
@@
 			(at 0 2.55 0)
 			(layer "F.Fab")
+			(hide yes)
 			(effects
 				(font
@@
 			(layer "F.Fab")
 		)
-		(fp_text user "${REFERENCE}"
-			(at 0 -2.45 0)
-			(layer "F.Fab")
-			(effects
-				(font
-					(size 1 1)
-					(thickness 0.15)
-				)
-			)
-		)
 		(pad "1" smd rect
 			(at -2.05 -0.8)
@@
 		(descr "LED SMD 0805 (2012 Metric), square (rectangular) end terminal, IPC-7351 nominal, (Body size source: https://docs.google.com/spreadsheets/d/1BsfQQcO9C6DZCsRaXUlFlo91Tg2WpOkGARC1WS5S8t0/edit?usp=sharing), generated with kicad-footprint-generator")
 		(tags "LED handsolder")
-		(property "Reference" "D3"
-			(at 0 -1.65 90)
+		(property "Reference" "BATT"
+			(at -3.319801 -0.0424 180)
 			(layer "F.SilkS")
 			(effects
@@
 			(at 0 1.65 90)
 			(layer "F.Fab")
+			(hide yes)
 			(effects
 				(font
@@
 			(at 0 -1.679999 0)
 			(layer "F.SilkS")
+			(hide yes)
 			(effects
 				(font
@@
 		(pad "2" smd roundrect
 			(at 3.149999 0 90)
-			(size 4 3.8)
+			(size 4 6)
 			(layers "F.Cu" "F.Mask" "F.Paste")
 			(roundrect_rratio 0.25)
@@
 			(at 2.9616 -0.06 0)
 			(layer "F.SilkS")
+			(hide yes)
 			(effects
 				(font
@@
 		(descr "LED SMD 0805 (2012 Metric), square (rectangular) end terminal, IPC-7351 nominal, (Body size source: https://docs.google.com/spreadsheets/d/1BsfQQcO9C6DZCsRaXUlFlo91Tg2WpOkGARC1WS5S8t0/edit?usp=sharing), generated with kicad-footprint-generator")
 		(tags "LED handsolder")
-		(property "Reference" "D2"
-			(at 0 -1.65 90)
+		(property "Reference" "3,3V"
+			(at -3.419801 -0.0184 180)
 			(layer "F.SilkS")
 			(effects
@@
 			(at 0 1.65 90)
 			(layer "F.Fab")
+			(hide yes)
 			(effects
 				(font
@@
 		(descr "CK components KMR2 tactile switch http://www.ckswitches.com/media/1479/kmr2.pdf")
 		(tags "tactile switch kmr2")
-		(property "Reference" "SW3"
+		(property "Reference" "STOP/GO"
 			(at 0 -2.450001 90)
 			(layer "F.SilkS")
@@
 			(layer "F.Fab")
 		)
-		(fp_text user "${REFERENCE}"
-			(at 0 -2.450001 90)
-			(layer "F.Fab")
-			(effects
-				(font
-					(size 1 1)
-					(thickness 0.15)
-				)
-			)
-		)
 		(pad "1" smd rect
 			(at -2.049999 -0.8 90)
@@
 			(at 0 -1.679999 0)
 			(layer "F.SilkS")
+			(hide yes)
 			(effects
 				(font
@@
 		(descr "CK components KMR2 tactile switch http://www.ckswitches.com/media/1479/kmr2.pdf")
 		(tags "tactile switch kmr2")
-		(property "Reference" "SW1"
-			(at 0 -2.45 0)
+		(property "Reference" "EN"
+			(at 0.000399 -2.359 0)
 			(layer "F.SilkS")
 			(effects
@@
 			(at 0 2.55 0)
 			(layer "F.Fab")
+			(hide yes)
 			(effects
 				(font
@@
 			(layer "F.Fab")
 		)
-		(fp_text user "${REFERENCE}"
-			(at 0 -2.45 0)
-			(layer "F.Fab")
-			(effects
-				(font
-					(size 1 1)
-					(thickness 0.15)
-				)
-			)
-		)
 		(pad "1" smd rect
 			(at -2.05 -0.8)
@@
 			(at 0 0 0)
 			(layer "B.SilkS")
+			(hide yes)
 			(effects
 				(font
@@
 	)
 	(via
+		(at 176.11 119.69)
+		(size 0.6)
+		(drill 0.3)
+		(layers "F.Cu" "B.Cu")
+		(free yes)
+		(net 1)
+	)
+	(via
 		(at 237.2145 152.247201)
 		(size 0.6)
@@
 	)
 	(segment
-		(start 242.7364 145.542001)
-		(end 242.7364 144.456704)
+		(start 241.023577 142.500029)
+		(end 241.016674 142.506932)
 		(width 0.75)
 		(layer "B.Cu")
@@
 	)
 	(segment
+		(start 230.644932 142.506932)
+		(end 230.638029 142.500029)
+		(width 0.75)
+		(layer "B.Cu")
+		(net 2)
+	)
+	(segment
+		(start 242.7364 145.542001)
+		(end 242.7364 144.456704)
+		(width 0.75)
+		(layer "B.Cu")
+		(net 2)
+	)
+	(segment
 		(start 157.964587 137.593786)
 		(end 160.8836 140.5128)
@@
 	)
 	(segment
-		(start 171.7548 158.75)
-		(end 193.38054 158.75)
+		(start 241.016674 142.506932)
+		(end 230.644932 142.506932)
 		(width 0.75)
 		(layer "B.Cu")
@@
 	)
 	(segment
-		(start 227.7872 145.3896)
-		(end 230.197776 142.979024)
+		(start 171.7548 158.75)
+		(end 193.38054 158.75)
 		(width 0.75)
 		(layer "B.Cu")
@@
 	)
 	(segment
-		(start 241.023577 142.500029)
-		(end 230.638029 142.500029)
+		(start 227.7872 145.3896)
+		(end 230.197776 142.979024)
 		(width 0.75)
 		(layer "B.Cu")
@@
 	)
 	(arc
+		(start 242.7364 144.456704)
+		(mid 242.574332 143.641931)
+		(end 242.1128 142.9512)
+		(width 0.75)
+		(layer "B.Cu")
+		(net 2)
+	)
+	(arc
 		(start 232.4608 130.550199)
 		(mid 232.758472 129.0537)
@@
 	)
 	(arc
-		(start 242.7364 144.456704)
-		(mid 242.574332 143.641931)
-		(end 242.1128 142.9512)
-		(width 0.75)
-		(layer "B.Cu")
-		(net 2)
-	)
-	(arc
 		(start 165.2016 152.49376)
 		(mid 165.716497 155.082323)
@@
 	)
 	(segment
+		(start 215.392 115.6716)
+		(end 215.383919 115.679681)
+		(width 0.3)
+		(layer "F.Cu")
+		(net 22)
+	)
+	(segment
 		(start 181.7624 114.373799)
 		(end 181.7624 110.082284)
@@
 	)
 	(segment
-		(start 234.734912 131.001312)
-		(end 222.242961 118.509361)
+		(start 196.248481 115.679681)
+		(end 196.2404 115.6716)
 		(width 0.3)
 		(layer "F.Cu")
@@
 	)
 	(segment
-		(start 215.392 115.6716)
-		(end 196.2404 115.6716)
+		(start 234.734912 131.001312)
+		(end 222.242961 118.509361)
 		(width 0.3)
 		(layer "F.Cu")
@@
 		(net 22)
 	)
+	(segment
+		(start 215.383919 115.679681)
+		(end 196.248481 115.679681)
+		(width 0.3)
+		(layer "F.Cu")
+		(net 22)
+	)
 	(via
 		(at 242.316 132.6896)
@@
 	)
 	(arc
-		(start 238.8108 132.6896)
-		(mid 236.604945 132.250828)
-		(end 234.734912 131.001312)
-		(width 0.3)
-		(layer "F.Cu")
-		(net 22)
-	)
-	(arc
 		(start 222.242961 118.509361)
 		(mid 219.099713 116.40911)
@@
 		(width 0.3)
 		(layer "F.Cu")
+		(net 22)
+	)
+	(arc
+		(start 238.8108 132.6896)
+		(mid 236.604945 132.250828)
+		(end 234.734912 131.001312)
+		(width 0.3)
+		(layer "F.Cu")
